File: X15_Brickstribution.sch (EAGLE design)
At the start: 77 parts, among them J1 IPL1-104-01-X-S-K, U5 IC_L4970A, U6 DIODE_STPS1545CT, U7 IC_L4970A, U8 DIODE_STPS1545CT

Commit message: In progress board
Parts:
- removed REV_TRANS: TRANS_IRF1018E_S_SLPBF, X15_Brickstribution:TRANS_IRF1018E_S_SLPBF
- added U$3: TRANS_IRF1018EPBF, X15_Brickstribution:TRANS_IRF1018EPBF
- renumbered R31 to R2
Connections:
- net +12V_CONV: no longer U5.VI, U7.VI
- net +48V: now also C1.1, C2.1, C3.1, U5.VI, U7.VI; no longer C1.2, C2.2, C3.2
- net 12V_GND: no longer 7.4V_GND.1, C23.1, C24.1, C26.1, C27.1, C28.1, C29.2, C30.1, C32.1, C33.1, C35.1, C36.1, C37.1, C38.2, C39.1, D12.C, D14.C, J1.03, J1.04, R23.1, R24.1, R26.1, R27.1, R28.1, R30.1, U5.GND, U5.RST, U6.1, U6.3, U7.GND, U7.RST, U8.1, U8.3
- net 48V_GND: now also 7.4V_GND.1, C1.2, C2.2, C23.1, C24.1, C26.1, C27.1, C28.1, C29.2, C3.2, C30.1, C32.1, C33.1, C35.1, C36.1, C37.1, C38.2, C39.1, D12.C, D14.C, J1.03, J1.04, R23.1, R24.1, R26.1, R27.1, R28.1, R30.1, U$3.S, U5.GND@1, U5.GND@2, U5.RST, U6.1, U6.3, U7.GND@1, U7.GND@2, U7.RST, U8.1, U8.3; no longer C1.1, C2.1, C3.1, REV_TRANS.S
- net GND_RAW: now also U$3.D; no longer REV_TRANS.D
- net REV_GATE: now also U$3.G; no longer REV_TRANS.G
Other:
- moved on the sheet: C1, C2, C3

Commit message: Alumni Revisions Implemented
Parts:
- removed D2: SK34A-TPDO-214AC_HSMA_MCC-M, X15_Brickstribution:SK34A-TPDO-214AC_HSMA_MCC-M
- removed D9: GREEN, SparkFun-LED:LED-GREEN0603
- removed R9: 470, SparkFun-Resistors:470OHM-0603-1/10W-1%
- added CR1: Zener, X15_Brickstribution:DIODE_SMBJ5357B-TPDIODE_DO-214AA_4P38X3P62_MCC-M
Connections:
- removed net +12V_CONV: +12V_TEST.1, BACKPLANE_CONN.07, BACKPLANE_POWER.VDD1, BACKPLANE_POWER.VDD2, BACKPLANE_POWER.VDD3, BACKPLANE_POWER.VDD4, BACKPLANE_POWER.VDD5, D2.1, R9.1, U$1.VIN+
- removed net N$8: D9.A, R9.2
- net +12V: now also +12V_TEST.1, BACKPLANE_CONN.07, BACKPLANE_POWER.VDD1, BACKPLANE_POWER.VDD2, BACKPLANE_POWER.VDD3, BACKPLANE_POWER.VDD4, BACKPLANE_POWER.VDD5, CR1.1, U$1.VIN+, U$1.VIN-; no longer D2.2
- net 12V_GND: now also CR1.2; no longer D9.C, U$1.VIN-
Other:
- note added: "Back EMF Diode"
- note removed: "ORing Diode to Conversion"
- moved on the sheet: D13, R22

Commit message: Final Iteration of Layout
Parts:
- removed D12: GREEN, SparkFun-LED:LED-GREEN0603
- removed D14: RED, SparkFun-LED:LED-RED0603
- removed R10: 150, SparkFun-Resistors:150OHM-0603-1/10W-1%
- removed R11: 100, SparkFun-Resistors:100OHM-0603-1/4W-5%
- removed R12, R21: 470, SparkFun-Resistors:470OHM-0603-1/10W-1%
- added D2, D3: Yellow, SparkFun-LED:LED-YELLOW0603
- added R3: 1.5k, SparkFun-Resistors:1.5KOHM-0603-1/10W-1%
- added R4: 100, SparkFun-Resistors:100OHM-0603-1/4W-5%
- added R5, R6: 150, SparkFun-Resistors:150OHM-0603-1/10W-1%
- R8: value 2.49k -> 20; device SparkFun-Resistors:2.49KOHM-0603-1/10W-1% -> SparkFun-Resistors:20OHM-0603-1/10W-1%
- renumbered R22 to R7
Connections:
- net +3.3V: now also R8.1; no longer R11.1
- net +48V: now also R3.1; no longer R8.1
- net +5V: now also R4.1; no longer R10.1
- net 48V_GND: now also D2.C, D3.C; no longer D12.C, D14.C
- net N$10: now also R8.2; no longer R11.2
- net N$11: now also D3.A, R6.2; no longer D14.A, R12.2
- net N$12: now also D2.A, R5.2; no longer D12.A, R21.2
- net N$4: now also R3.2; no longer R8.2
- net N$9: now also R4.2; no longer R10.2
- net VOUT1: now also R5.1; no longer R21.1
- net VOUT2: now also R6.1; no longer R12.1
Other:
- moved on the sheet: R8

Commit message: Revision before implementing Samtec Brick Connectors
Parts:
- C1, C2, C3: value 0.330mF -> 330uF; device X15_Brickstribution:EMZR500ADA331MJA0GCAP_MZR_JA0_NIP-M -> X15_Brickstribution:CAP_MAL215099112E3CAP_099112E3_VIS-M
- CR1: value Zener -> DIODE(Z)_SMBJ5357B-TPDIODE_DO-214AA_4P38X3P62_MCC-M; device X15_Brickstribution:DIODE_SMBJ5357B-TPDIODE_DO-214AA_4P38X3P62_MCC-M -> X15_Brickstribution:DIODE(Z)_SMBJ5357B-TPDIODE_DO-214AA_4P38X3P62_MCC-M
- U$3: value TRANS_IRF1018EPBF -> TRANS_IRF1018ESTRLPBF
